Commit message: Working launch with both Robots

File: catkin_ws/src/cell_support/urdf/cell.xacro (robot description, xacro)
@@ -1,19 +1,20 @@
 <?xml version="1.0" ?>
-<robot name="cell" xmlns:xacro="https://ros.org/wiki/xarco">
+<robot name="cell" xmlns:xacro="https://ros.org/wiki/xacro">
  <xacro:include filename="$(find ur_description)/urdf/ur3.urdf.xacro"/>
- <xacro:include filename="$(find abb_experimental)/abb_irb120_support/urdf/irb120.xacro"/>
+ <xacro:include filename="$(find abb_irb120_support)/urdf/irb120_macro.xacro"/>
   <link name="world"/>
-  <!-- instantiating arm  -->
-  <xacro:ur3_robot prefix="" joint_limited="true"/>
-  <xacro:abb_irb120 prefix="" />
-  <joint name="world_to_ur3" type="fixed">
+  <!-- init robots -->
+  <xacro:ur3_robot prefix="ur3_" joint_limited="true"/>
+  <xacro:abb_irb120 prefix="irb120_" />
+  <!-- Joints -->
+  <joint name="world_to_UR3" type="fixed">
     <parent link="world"/>
-    <child link="base_link"/>
+    <child link="ur3_base_link"/>
     <origin xyz="0 0 0" rpy="0 0 0" />
   </joint>
   <joint name="world_to_irb120" type="fixed">
     <parent link="world" />
-    <child link="base_link"/>
-    <origin xyz="0.1 0.1 0" rpy="0 0 0"/>
+    <child link="irb120_base_link"/>
+    <origin xyz="1 0 0" rpy="0 0 0"/>
   </joint>
 </robot>
