Commit message: Added Launchfiles for all three

File: catkin_ws/src/cell_support/urdf/cell_both.xacro (robot description, xacro)
@@ -16,5 +16,5 @@
     <parent link="world" />
     <child link="irb120_base_link"/>
-    <origin xyz="1 0 0" rpy="0 0 0"/>
+    <origin xyz="0 1 0" rpy="0 0 0"/>
   </joint>
 </robot>
