Commit message: To many updates

File: src/cell_support/urdf/unterbau.xacro (robot description, xacro)
@@ -7,5 +7,5 @@
             <origin rpy="0 0 1.57" xyz="-1.075 0.023 -0.021" />
             <geometry>
-               <mesh filename="package://cell_support/meshes/Mittelteil_noRobot.stl" scale="0.001 0.001 0.001"/>
+               <mesh filename="package://cell_support/meshes/1000_Industrie_4_0_Demonstrator.stl" scale="0.001 0.001 0.001"/>
             </geometry>
          </visual>
