Commit message: Added Moveit for irb120 with gripper

File: src/cell_support/urdf/cell_irb120.xacro (robot description, xacro)
@@ -16,5 +16,5 @@
     <parent link="irb120_tool0" />
     <child link="gripper_frame" />
-    <origin xyz="0 0 0" rpy="0 0 0" />
+    <origin xyz="0 0 0" rpy="0 1.57 0" />
   </joint>
 </robot>

File: src/cell_support/urdf/gripper.xacro (robot description, xacro)
@@ -2,9 +2,10 @@
 <robot xmlns:xacro="http://ros.org/wiki/xacro">
   <xacro:macro name="gripper_definition" params="prefix">
+    <link name="${prefix}gripper_tool" />
     <link name="${prefix}gripper_body">
       <visual>
-        <origin xyz="0.1 0 0" rpy="0 0 0" />
+        <origin xyz="0 0 -0.005" rpy="0 0 0" />
         <geometry>
-          <mesh filename="package://cell_support/meshes/gripper.dae"/>
+          <mesh filename="package://cell_support/meshes/4003_Greifer_Roboter.stl" scale="0.001 0.001 0.001"/>
         </geometry>
         <material name="">
@@ -13,7 +14,7 @@
       </visual>
       <collision>
-        <origin xyz="0.0575 0 0" rpy="0 0 0" />
+        <origin xyz="0 0 0.0575" rpy="0 0 0" />
         <geometry>
-          <box size="0.115 0.052 0.052" />
+          <box size="0.052 0.052 0.115" />
         </geometry>
         <material name="yellow">
@@ -42,4 +43,9 @@
       <origin xyz="0 0 0" rpy="0 0 0" />
     </joint>
+    <joint name="body_to_tool" type="fixed">
+      <parent link="${prefix}gripper_body" />
+      <child link="${prefix}gripper_tool" />
+      <origin xyz="0 0 0.155" rpy="0 0 0" />
+    </joint>
   </xacro:macro>
 </robot>

Commit message: Multiple Structural Updates

File: src/cell_support/urdf/cell_irb120.xacro (robot description, xacro)
@@ -3,12 +3,19 @@
  <xacro:include filename="$(find abb_irb120_support)/urdf/irb120_macro.xacro"/>
  <xacro:include filename="$(find cell_support)/urdf/gripper.xacro" />
+ <xacro:include filename="$(find cell_support)/urdf/cell_base.xacro" />
   <link name="world"/>
   <!-- init robots -->
   <xacro:abb_irb120 prefix="irb120_" />
   <xacro:gripper_definition prefix="" />
+  <xacro:cell_base prefix=""/>
   <!-- Joints -->
   <joint name="world_to_irb120" type="fixed">
     <parent link="world" />
     <child link="irb120_base_link"/>
+    <origin xyz="0 0 0" rpy="0 0 0"/>
+  </joint>
+    <joint name="world_to_cellBase" type="fixed">
+    <parent link="world" />
+    <child link="base"/>
     <origin xyz="0 0 0" rpy="0 0 0"/>
   </joint>

File: src/cell_support/urdf/gripper.xacro (robot description, xacro)
@@ -1,4 +1,4 @@
 <?xml version="1.0" encoding="UTF-8"?>
-<robot xmlns:xacro="http://ros.org/wiki/xacro1">
+<robot xmlns:xacro="https://ros.org/wiki/xacro">
   <xacro:macro name="gripper_definition" params="prefix">
     <link name="${prefix}gripper_tool">

Commit message: Added Staubli tx2-60l

File: src/cell_support/urdf/cell_irb120.xacro (robot description, xacro)
@@ -4,5 +4,5 @@
  <xacro:include filename="$(find cell_support)/urdf/gripper.xacro" />
  <xacro:include filename="$(find cell_support)/urdf/cell_base.xacro" />
-  <link name="world"/>
+  <link name="root_link"/>
   <!-- init robots -->
   <xacro:abb_irb120 prefix="irb120_" />
@@ -10,12 +10,12 @@
   <xacro:cell_base prefix=""/>
   <!-- Joints -->
-  <joint name="world_to_irb120" type="fixed">
-    <parent link="world" />
+  <joint name="cell_base_to_irb120" type="fixed">
+    <parent link="cell_base" />
     <child link="irb120_base_link"/>
     <origin xyz="0 0 0" rpy="0 0 0"/>
   </joint>
     <joint name="world_to_cellBase" type="fixed">
-    <parent link="world" />
-    <child link="base"/>
+    <parent link="root_link" />
+    <child link="cell_base"/>
     <origin xyz="0 0 0" rpy="0 0 0"/>
   </joint>

Commit message: Test Update

File: src/cell_support/urdf/cell_irb120.xacro (robot description, xacro)
@@ -2,14 +2,14 @@
 <robot name="cell" xmlns:xacro="https://ros.org/wiki/xacro">
  <xacro:include filename="$(find abb_irb120_support)/urdf/irb120_macro.xacro"/>
- <xacro:include filename="$(find cell_support)/urdf/gripper.xacro" />
- <xacro:include filename="$(find cell_support)/urdf/cell_base.xacro" />
+ <xacro:include filename="$(find cell_support)/urdf/gripper_definition.xacro" />
+ <xacro:include filename="$(find cell_support)/urdf/unterbau.xacro" />
   <link name="root_link"/>
   <!-- init robots -->
   <xacro:abb_irb120 prefix="irb120_" />
   <xacro:gripper_definition prefix="" />
-  <xacro:cell_base prefix=""/>
+  <xacro:unterbau prefix=""/>
   <!-- Joints -->
   <joint name="cell_base_to_irb120" type="fixed">
-    <parent link="cell_base" />
+    <parent link="root_link" />
     <child link="irb120_base_link"/>
     <origin xyz="0 0 0" rpy="0 0 0"/>
@@ -17,5 +17,5 @@
     <joint name="world_to_cellBase" type="fixed">
     <parent link="root_link" />
-    <child link="cell_base"/>
+    <child link="unterbau_base"/>
     <origin xyz="0 0 0" rpy="0 0 0"/>
   </joint>

File: src/cell_support/urdf/unterbau.xacro (robot description, xacro)
@@ -1,7 +1,7 @@
 <?xml version="1.0" encoding="UTF-8"?>
 <robot xmlns:xacro="https://ros.org/wiki/xacro">
-   <xacro:macro name="plant" params="prefix">
-      <link name="plant_base" />
-      <link name="plant_body">
+   <xacro:macro name="unterbau" params="prefix">
+      <link name="unterbau_base" />
+      <link name="unterbau_body">
          <visual>
             <origin rpy="0 0 1.57" xyz="-1.075 0.023 -0.021" />
@@ -18,6 +18,6 @@
       </link>
       <joint name="base_to_body" type="fixed">
-        <parent link="plant_base" />
-        <child link="plant_body" />
+        <parent link="unterbau_base" />
+        <child link="unterbau_body" />
         <origin xyz="0 0 0" rpy="0 0 0" />
       </joint>

Commit message: Working Cell

File: src/cell_support/urdf/cell_irb120.xacro (robot description, xacro)
@@ -1,27 +1,20 @@
 <?xml version="1.0" ?>
-<robot name="cell" xmlns:xacro="https://ros.org/wiki/xacro">
- <xacro:include filename="$(find abb_irb120_support)/urdf/irb120_macro.xacro"/>
- <xacro:include filename="$(find cell_support)/urdf/gripper_definition.xacro" />
+<robot name="cell_irb120" xmlns:xacro="https://ros.org/wiki/xacro">
+ <xacro:include filename="$(find cell_support)/urdf/irb120_gripper.xacro"/>
  <xacro:include filename="$(find cell_support)/urdf/unterbau.xacro" />
   <link name="root_link"/>
   <!-- init robots -->
-  <xacro:abb_irb120 prefix="irb120_" />
-  <xacro:gripper_definition prefix="" />
+  <xacro:irb120_gripper />
   <xacro:unterbau prefix=""/>
   <!-- Joints -->
-  <joint name="cell_base_to_irb120" type="fixed">
+  <joint name="root_to_irb120" type="fixed">
     <parent link="root_link" />
     <child link="irb120_base_link"/>
     <origin xyz="0 0 0" rpy="0 0 0"/>
   </joint>
-    <joint name="world_to_cellBase" type="fixed">
+  <joint name="root_to_unterbau" type="fixed">
     <parent link="root_link" />
     <child link="unterbau_base"/>
     <origin xyz="0 0 0" rpy="0 0 0"/>
   </joint>
-  <joint name="tool0_to_gripper" type="fixed">
-    <parent link="irb120_tool0" />
-    <child link="gripper_frame" />
-    <origin xyz="0 0 0" rpy="0 1.57 0" />
-  </joint>
 </robot>

File: src/cell_support/urdf/cell_irb120_generated.urdf (robot description, URDF)
Before this commit: robot cell, 15 links, 14 joints
Joints:
- removed joint cell_base_to_irb120
- removed joint world_to_cellBase
- added joint root_to_irb120: type fixed, parent root_link, child irb120_base_link, origin xyz=0 0 0 rpy=0 0 0
- added joint root_to_unterbau: type fixed, parent root_link, child unterbau_base, origin xyz=0 0 0 rpy=0 0 0

File: src/cell_support/urdf/unterbau.xacro (robot description, xacro)
@@ -3,5 +3,5 @@
    <xacro:macro name="unterbau" params="prefix">
       <link name="unterbau_base" />
-      <link name="unterbau_body">
+     <link name="unterbau_body">
          <visual>
             <origin rpy="0 0 1.57" xyz="-1.075 0.023 -0.021" />
@@ -13,5 +13,5 @@
             <origin rpy="0 0 1.57" xyz="-1.075 0.023 -0.021" />
             <geometry>
-               <mesh filename="package://cell_support/meshes/Mittelteil_noRobot.stl" scale="0.001 0.001 0.001"/>
+               <mesh filename="package://cell_support/meshes/Mittelteil_final_collision.stl" scale="0.001 0.001 0.001"/>
             </geometry>
          </collision>

Commit message: Minor bugfix

File: src/cell_support/urdf/cell_irb120.xacro (robot description, xacro)
@@ -3,5 +3,5 @@
  <xacro:include filename="$(find cell_support)/urdf/irb120_gripper.xacro"/>
  <xacro:include filename="$(find cell_support)/urdf/unterbau.xacro" />
-  <link name="root_link"/>
+  <link name="world"/>
   <!-- init robots -->
   <xacro:irb120_gripper />
@@ -9,10 +9,10 @@
   <!-- Joints -->
   <joint name="root_to_irb120" type="fixed">
-    <parent link="root_link" />
+    <parent link="world" />
     <child link="irb120_base_link"/>
     <origin xyz="0 0 0" rpy="0 0 0"/>
   </joint>
   <joint name="root_to_unterbau" type="fixed">
-    <parent link="root_link" />
+    <parent link="world" />
     <child link="unterbau_base"/>
     <origin xyz="0 0 0" rpy="0 0 0"/>

File: src/cell_support/urdf/unterbau.xacro (robot description, xacro)
@@ -7,5 +7,5 @@
             <origin rpy="0 0 1.57" xyz="-1.075 0.023 -0.021" />
             <geometry>
-               <mesh filename="package://cell_support/meshes/1000_Industrie_4_0_Demonstrator.stl" scale="0.001 0.001 0.001"/>
+               <mesh filename="package://cell_support/meshes/Mittelteil_final_collision.stl" scale="0.001 0.001 0.001"/>
             </geometry>
          </visual>

Commit message: Diverses

File: src/cell_support/urdf/cell_irb120.xacro (robot description, xacro)
@@ -1,15 +1,22 @@
 <?xml version="1.0" ?>
 <robot name="cell_irb120" xmlns:xacro="https://ros.org/wiki/xacro">
- <xacro:include filename="$(find cell_support)/urdf/irb120_gripper.xacro"/>
+ <xacro:include filename="$(find cell_support)/urdf/gripper_definition.xacro"/>
  <xacro:include filename="$(find cell_support)/urdf/unterbau.xacro" />
+ <xacro:include filename="$(find abb_irb120_support)/urdf/irb120_macro.xacro" />
   <link name="world"/>
-  <!-- init robots -->
-  <xacro:irb120_gripper />
-  <xacro:unterbau prefix=""/>
+  <!-- init -->
+  <xacro:gripper_definition prefix="" />
+  <xacro:unterbau prefix="" />
+  <xacro:abb_irb120 prefix="" />
   <!-- Joints -->
   <joint name="root_to_irb120" type="fixed">
     <parent link="world" />
-    <child link="irb120_base_link"/>
+    <child link="base_link"/>
     <origin xyz="0 0 0" rpy="0 0 0"/>
+  </joint>
+  <joint name="tool0_to_gripper" type="fixed">
+    <parent link="tool0" />
+    <child link="gripper_frame" />
+    <origin xyz="0 0 0" rpy="0 1.57 0" />
   </joint>
   <joint name="root_to_unterbau" type="fixed">

File: src/cell_support/urdf/cell_tx260l.xacro (robot description, xacro)
@@ -1,20 +1,27 @@
 <?xml version="1.0" ?>
 <robot name="cell_tx260l" xmlns:xacro="https://ros.org/wiki/xacro">
- <xacro:include filename="$(find cell_support)/urdf/tx260l_gripper.xacro"/>
+ <xacro:include filename="$(find cell_support)/urdf/gripper_definition.xacro"/>
  <xacro:include filename="$(find cell_support)/urdf/unterbau.xacro" />
-  <link name="root_link"/>
+ <xacro:include filename="$(find staubli_tx260l_support)/urdf/tx60l_macro.xacro"/>
+  <link name="world"/>
   <!-- init robots -->
-  <xacro:tx260l_gripper />
+  <xacro:gripper_definition prefix="" />
   <xacro:unterbau prefix=""/>
+  <xacro:staubli_tx260l prefix="" />
   <!-- Joints -->
-  <joint name="root_to_tx260l" type="fixed">
-    <parent link="root_link" />
-    <child link="tx260l_base_link"/>
+  <joint name="world_to_tx260l" type="fixed">
+    <parent link="world" />
+    <child link="base_link"/>
     <origin xyz="0 0 0" rpy="0 0 0"/>
   </joint>
-  <joint name="root_to_unterbau" type="fixed">
-    <parent link="root_link" />
+  <joint name="world_to_unterbau" type="fixed">
+    <parent link="world" />
     <child link="unterbau_base"/>
     <origin xyz="0 0 0" rpy="0 0 0"/>
   </joint>
+  <joint name="tool0_to_gripper" type="fixed">
+    <parent link="tool0" />
+    <child link="gripper_frame" />
+    <origin xyz="0 0 0" rpy="0 1.57 0" />
+  </joint>
 </robot>

File: src/cell_support/urdf/cell_ur3.xacro (robot description, xacro)
@@ -5,4 +5,6 @@
   <!-- init robots -->
   <xacro:ur3_robot prefix="ur3_" joint_limited="true"/>
+  <xacro:unterbau prefix="" />
+  <xacro:gripper_definition prefix="" />
   <!-- Joints -->
   <joint name="world_to_UR3" type="fixed">
@@ -11,3 +13,13 @@
     <origin xyz="0 0 0" rpy="0 0 0" />
   </joint>
+  <joint name="tool0_to_gripper" type="fixed">
+    <parent link="tool0" />
+    <child link="gripper_frame" />
+    <origin xyz="0 0 0" rpy="0 1.57 0" />
+  </joint>
+  <joint name="world_to_unterbau" type="fixed">
+    <parent link="world" />
+    <child link="unterbau_base"/>
+    <origin xyz="0 0 0" rpy="0 0 0"/>
+  </joint>
 </robot>

File: src/cell_support/urdf/gripper_definition.xacro (robot description, xacro)
@@ -2,6 +2,6 @@
 <robot xmlns:xacro="https://ros.org/wiki/xacro">
   <xacro:macro name="gripper_definition" params="prefix">
-    <link name="${prefix}gripper_tool">
-          <visual>
+    <link name="${prefix}grasping_frame">
+      <visual>
         <geometry>
           <sphere radius="0.005" />
@@ -11,5 +11,5 @@
         </material>
       </visual>
-      </link>
+    </link>
     <link name="${prefix}gripper_body">
       <visual>
@@ -54,5 +54,5 @@
     <joint name="body_to_tool" type="fixed">
       <parent link="${prefix}gripper_body" />
-      <child link="${prefix}gripper_tool" />
+      <child link="${prefix}grasping_frame" />
       <origin xyz="0 0 0.155" rpy="0 0 0" />
     </joint>

File: src/cell_support/urdf/unterbau.xacro (robot description, xacro)
@@ -7,11 +7,13 @@
             <origin rpy="0 0 1.57" xyz="-1.075 0.023 -0.021" />
             <geometry>
-               <mesh filename="package://cell_support/meshes/Mittelteil_final_collision.stl" scale="0.001 0.001 0.001"/>
+               <mesh filename="package://cell_support/meshes/1000_Industrie_4_0_Demonstrator_V2.stl" scale="0.001 0.001 0.001"/>
             </geometry>
          </visual>
-         <collision>
-            <origin rpy="0 0 1.57" xyz="-1.075 0.023 -0.021" />
-            <geometry>
-               <mesh filename="package://cell_support/meshes/Mittelteil_final_collision.stl" scale="0.001 0.001 0.001"/>
+        <collision>
+          <!-- origin rpy="0 0 1.57" xyz="-1.075 0.023 -0.021" /-->
+          <origin rpy="0 0 0" xyz="0 0 0.005" />
+          <geometry>
+            <sphere radius="0.0001" />
+               <!-- mesh filename="package://cell_support/meshes/Mittelteil_final_collision.stl" scale="0.001 0.001 0.001"/ -->
             </geometry>
          </collision>

Commit message: Updated Collision

File: src/cell_support/urdf/cell_irb120.xacro (robot description, xacro)
@@ -17,5 +17,5 @@
   <joint name="tool0_to_gripper" type="fixed">
     <parent link="tool0" />
-    <child link="gripper_frame" />
+    <child link="gripper_base" />
     <origin xyz="0 0 0" rpy="0 1.57 0" />
   </joint>

File: src/cell_support/urdf/cell_tx260l.xacro (robot description, xacro)
@@ -22,5 +22,5 @@
   <joint name="tool0_to_gripper" type="fixed">
     <parent link="tool0" />
-    <child link="gripper_frame" />
+    <child link="gripper_base" />
     <origin xyz="0 0 0" rpy="0 1.57 0" />
   </joint>

File: src/cell_support/urdf/gripper_definition.xacro (robot description, xacro)
@@ -5,5 +5,20 @@
       <visual>
         <geometry>
-          <sphere radius="0.005" />
+          <sphere radius="0.002" />
+        </geometry>
+        <material name="white">
+          <color rgba="1 1 1 0.5" />
+        </material>
+      </visual>
+      <collision>
+        <geometry>
+          <sphere radius="0.00000001" />
+        </geometry>
+      </collision>
+    </link>
+        <link name="${prefix}small_grasping_frame">
+      <visual>
+        <geometry>
+          <sphere radius="0.002" />
         </geometry>
         <material name="white">
@@ -19,7 +34,7 @@
     <link name="${prefix}gripper_body">
       <visual>
-        <origin xyz="0 0 -0.005" rpy="0 0 0" />
+        <origin xyz="0 0 0" rpy="0 0 0" />
         <geometry>
-          <mesh filename="package://cell_support/meshes/4003_Greifer_Roboter.stl" scale="0.001 0.001 0.001"/>
+          <mesh filename="package://cell_support/meshes/4003_Greifer_visual.stl" scale="0.001 0.001 0.001"/>
         </geometry>
         <material name="">
@@ -28,7 +43,7 @@
       </visual>
       <collision>
-        <origin xyz="0 0 -0.005" rpy="0 0 0" />
+        <origin xyz="0 0 0" rpy="0 0 0" />
         <geometry>
-          <mesh filename="package://cell_support/meshes/4003_Greifer_Roboter.stl" scale="0.001 0.001 0.001"/>
+          <mesh filename="package://cell_support/meshes/4003_Greifer_collision.stl" scale="0.001 0.001 0.001"/>
         </geometry>
         <material name="yellow">
@@ -37,5 +52,5 @@
       </collision>
     </link>
-    <link name="gripper_frame">
+    <link name="${prefix}gripper_base">
       <visual>
         <geometry>
@@ -52,13 +67,18 @@
       </collision>
     </link>
-    <joint name="body_to_frame" type="fixed">
-      <parent link="gripper_frame" />
-      <child link="gripper_body" />
+    <joint name="body_to_base" type="fixed">
+      <parent link="${prefix}gripper_base" />
+      <child link="${prefix}gripper_body" />
       <origin xyz="0 0 0" rpy="0 0 -0.785" />
     </joint>
-    <joint name="body_to_tool" type="fixed">
-      <parent link="${prefix}gripper_body" />
+    <joint name="frame_to_base" type="fixed">
+      <parent link="${prefix}gripper_base" />
       <child link="${prefix}grasping_frame" />
-      <origin xyz="0 0 0.155" rpy="0 0 0" />
+      <origin xyz="0 0 0.17225" rpy="0 0 -0.785" />
+    </joint>
+    <joint name="smallframe_to_base" type="fixed">
+      <parent link="${prefix}gripper_base" />
+      <child link="${prefix}small_grasping_frame" />
+      <origin xyz="0 0 0.16425" rpy="0 0 -0.785" />
     </joint>
   </xacro:macro>

File: src/cell_support/urdf/unterbau.xacro (robot description, xacro)
@@ -7,5 +7,5 @@
             <origin rpy="0 0 1.57" xyz="-1.075 0.023 -0.021" />
             <geometry>
-               <mesh filename="package://cell_support/meshes/1000_Industrie_4_0_Demonstrator_V2.stl" scale="0.001 0.001 0.001"/>
+               <mesh filename="package://cell_support/meshes/1000_Anlage_visual.stl" scale="0.001 0.001 0.001"/>
             </geometry>
          </visual>
@@ -15,5 +15,5 @@
           <geometry>
             <sphere radius="0.0001" />
-               <!-- mesh filename="package://cell_support/meshes/Mittelteil_final_collision.stl" scale="0.001 0.001 0.001"/ -->
+            <!--mesh filename="package://cell_support/meshes/1000_Anlage_collision.stl" scale="0.001 0.001 0.001" /-->
             </geometry>
          </collision>
