Commit message: Div Anpassungen

File: src/cell_support/urdf/gripper_definition.xacro (robot description, xacro)
@@ -11,4 +11,9 @@
         </material>
       </visual>
+      <collision>
+        <geometry>
+          <sphere radius="0.00000001" />
+        </geometry>
+      </collision>
     </link>
     <link name="${prefix}gripper_body">

Commit message: Div Updates

File: src/cell_support/urdf/gripper_definition.xacro (robot description, xacro)
@@ -55,5 +55,5 @@
       <parent link="gripper_frame" />
       <child link="gripper_body" />
-      <origin xyz="0 0 0" rpy="0 0 0" />
+      <origin xyz="0 0 0" rpy="0 0 -0.785" />
     </joint>
     <joint name="body_to_tool" type="fixed">

Commit message: removed small bug

File: src/cell_support/urdf/gripper_definition.xacro (robot description, xacro)
@@ -17,5 +17,5 @@
       </collision>
     </link>
-        <link name="${prefix}small_grasping_frame">
+    <link name="${prefix}small_grasping_frame">
       <visual>
         <geometry>
