Commit message: Adding Gripper

File: src/abb_experimental/abb_irb120_support/urdf/irb120.urdf (robot description, URDF)
Before this commit: robot abb_irb120, 9 links, 8 joints
Joints:
- joint joint_6: limit lower=-6.98132 upper=6.98132 effort=0 velocity=7.33038 -> lower=-3.2 upper=3.2 effort=0 velocity=7.33038

File: src/cell_support/urdf/cell_irb120.xacro (robot description, xacro)
@@ -2,7 +2,9 @@
 <robot name="cell" xmlns:xacro="https://ros.org/wiki/xacro">
  <xacro:include filename="$(find abb_irb120_support)/urdf/irb120_macro.xacro"/>
+ <xacro:include filename="$(find cell_support)/urdf/gripper.xacro" />
   <link name="world"/>
   <!-- init robots -->
   <xacro:abb_irb120 prefix="irb120_" />
+  <xacro:gripper_definition prefix="" />
   <!-- Joints -->
   <joint name="world_to_irb120" type="fixed">
@@ -11,3 +13,8 @@
     <origin xyz="0 0 0" rpy="0 0 0"/>
   </joint>
+  <joint name="tool0_to_gripper" type="fixed">
+    <parent link="irb120_tool0" />
+    <child link="gripper_frame" />
+    <origin xyz="0 0 0" rpy="0 0 0" />
+  </joint>
 </robot>
