Commit message: FIX Staubli

File: src/staubli_experimental/staubli_tx260l_support/urdf/tx60l_macro.xacro (robot description, xacro)
@@ -8,12 +8,12 @@
             <origin xyz="0 0 0" rpy="0 0 0" />
             <geometry>
-               <mesh filename="package://staubli_tx260l_support/meshes/tx60l/visual/base_link.stl" />
-            </geometry>
-            <xacro:material_staubli_ral_melon_yellow />
-         </visual>
-         <collision>
-            <origin xyz="0 0 0" rpy="0 0 0" />
-            <geometry>
-               <mesh filename="package://staubli_tx260l_support/meshes/tx60l/collision/base_link.stl" />
+               <mesh filename="package://staubli_tx260l_support/meshes/tx260l/visual/base_link.stl" />
+            </geometry>
+            <xacro:material_staubli_ral_melon_yellow />
+         </visual>
+         <collision>
+            <origin xyz="0 0 0" rpy="0 0 0" />
+            <geometry>
+               <mesh filename="package://staubli_tx260l_support/meshes/tx260l/collision/base_link.stl" />
             </geometry>
          </collision>
@@ -28,12 +28,12 @@
             <origin xyz="0 0 0" rpy="0 0 0" />
             <geometry>
-               <mesh filename="package://staubli_tx260l_support/meshes/tx60l/visual/link_1.stl" />
-            </geometry>
-            <xacro:material_staubli_ral_melon_yellow />
-         </visual>
-         <collision>
-            <origin xyz="0 0 0" rpy="0 0 0" />
-            <geometry>
-               <mesh filename="package://staubli_tx260l_support/meshes/tx60l/collision/link_1.stl" />
+               <mesh filename="package://staubli_tx260l_support/meshes/tx260l/visual/link_1.stl" />
+            </geometry>
+            <xacro:material_staubli_ral_melon_yellow />
+         </visual>
+         <collision>
+            <origin xyz="0 0 0" rpy="0 0 0" />
+            <geometry>
+               <mesh filename="package://staubli_tx260l_support/meshes/tx260l/collision/link_1.stl" />
             </geometry>
          </collision>
@@ -48,12 +48,12 @@
             <origin xyz="0 0 0" rpy="0 0 0" />
             <geometry>
-               <mesh filename="package://staubli_tx260l_support/meshes/tx60l/visual/link_2.stl" />
-            </geometry>
-            <xacro:material_staubli_ral_melon_yellow />
-         </visual>
-         <collision>
-            <origin xyz="0 0 0" rpy="0 0 0" />
-            <geometry>
-               <mesh filename="package://staubli_tx260l_support/meshes/tx60l/collision/link_2.stl" />
+               <mesh filename="package://staubli_tx260l_support/meshes/tx260l/visual/link_2.stl" />
+            </geometry>
+            <xacro:material_staubli_ral_melon_yellow />
+         </visual>
+         <collision>
+            <origin xyz="0 0 0" rpy="0 0 0" />
+            <geometry>
+               <mesh filename="package://staubli_tx260l_support/meshes/tx260l/collision/link_2.stl" />
             </geometry>
          </collision>
@@ -68,12 +68,12 @@
             <origin xyz="0 0 0" rpy="0 0 0" />
             <geometry>
-               <mesh filename="package://staubli_tx260l_support/meshes/tx60l/visual/link_3.stl" />
-            </geometry>
-            <xacro:material_staubli_ral_melon_yellow />
-         </visual>
-         <collision>
-            <origin xyz="0 0 0" rpy="0 0 0" />
-            <geometry>
-               <mesh filename="package://staubli_tx260l_support/meshes/tx60l/collision/link_3.stl" />
+               <mesh filename="package://staubli_tx260l_support/meshes/tx260l/visual/link_3.stl" />
+            </geometry>
+            <xacro:material_staubli_ral_melon_yellow />
+         </visual>
+         <collision>
+            <origin xyz="0 0 0" rpy="0 0 0" />
+            <geometry>
+               <mesh filename="package://staubli_tx260l_support/meshes/tx260l/collision/link_3.stl" />
             </geometry>
          </collision>
@@ -88,12 +88,12 @@
             <origin xyz="0 0 0" rpy="0 0 0" />
             <geometry>
-               <mesh filename="package://staubli_tx260l_support/meshes/tx60l/visual/link_4.stl" />
-            </geometry>
-            <xacro:material_staubli_ral_melon_yellow />
-         </visual>
-         <collision>
-            <origin xyz="0 0 0" rpy="0 0 0" />
-            <geometry>
-               <mesh filename="package://staubli_tx260l_support/meshes/tx60l/collision/link_4.stl" />
+               <mesh filename="package://staubli_tx260l_support/meshes/tx260l/visual/link_4.stl" />
+            </geometry>
+            <xacro:material_staubli_ral_melon_yellow />
+         </visual>
+         <collision>
+            <origin xyz="0 0 0" rpy="0 0 0" />
+            <geometry>
+               <mesh filename="package://staubli_tx260l_support/meshes/tx260l/collision/link_4.stl" />
             </geometry>
          </collision>
@@ -108,5 +108,5 @@
             <origin xyz="0 0 0" rpy="0 0 0" />
             <geometry>
-               <mesh filename="package://staubli_tx260l_support/meshes/tx60l/visual/link_5.stl" />
+               <mesh filename="package://staubli_tx260l_support/meshes/tx260l/visual/link_5.stl" />
             </geometry>
             <xacro:material_staubli_ral_grey_aluminium />
@@ -115,5 +115,5 @@
             <origin xyz="0 0 0" rpy="0 0 0" />
             <geometry>
-               <mesh filename="package://staubli_tx260l_support/meshes/tx60l/collision/link_5.stl" />
+               <mesh filename="package://staubli_tx260l_support/meshes/tx260l/collision/link_5.stl" />
             </geometry>
          </collision>
@@ -128,5 +128,5 @@
             <origin xyz="0 0 0" rpy="0 0 0" />
             <geometry>
-               <mesh filename="package://staubli_tx260l_support/meshes/tx60l/visual/link_6.stl" />
+               <mesh filename="package://staubli_tx260l_support/meshes/tx260l/visual/link_6.stl" />
             </geometry>
             <xacro:material_staubli_ral_grey_aluminium />
@@ -135,5 +135,5 @@
             <origin xyz="0 0 0" rpy="0 0 0" />
             <geometry>
-               <mesh filename="package://staubli_tx260l_support/meshes/tx60l/collision/link_6.stl" />
+               <mesh filename="package://staubli_tx260l_support/meshes/tx260l/collision/link_6.stl" />
             </geometry>
          </collision>
